Commit message: modify urdf. minicheetah 2m/s finetuning

File: rsc/mini_cheetah/mini-cheetah-vision-v1.3.urdf (robot description, URDF)
Before this commit: robot mini_cheetah, 17 links, 16 joints
Links:
- link thigh_fl: geometry collision box size=0.025 0.025 0.16; visual mesh filename=meshes/mini_upper_link.obj
- link thigh_fr: geometry collision box size=0.025 0.025 0.16; visual mesh filename=meshes/mini_upper_link.obj
- link thigh_hl: geometry collision box size=0.025 0.025 0.16; visual mesh filename=meshes/mini_upper_link.obj
- link thigh_hr: geometry collision box size=0.025 0.025 0.16; visual mesh filename=meshes/mini_upper_link.obj
Joints:
- joint abduct_fl_to_thigh_fl_j: limit lower=-4.712388 upper=4.712388 velocity=40 -> lower=-4.712388 upper=4.712388 effort=18 velocity=40
- joint abduct_fr_to_thigh_fr_j: limit lower=-4.712388 upper=4.712388 velocity=40 -> lower=-4.712388 upper=4.712388 effort=18 velocity=40
- joint abduct_hl_to_thigh_hl_j: limit lower=-4.712388 upper=4.712388 velocity=40 -> lower=-4.712388 upper=4.712388 effort=18 velocity=40
- joint abduct_hr_to_thigh_hr_j: limit lower=-4.712388 upper=4.712388 velocity=40 -> lower=-4.712388 upper=4.712388 effort=18 velocity=40
- joint thigh_fl_to_knee_fl_j: limit lower=-2.705259778 upper=2.705259778 -> lower=-2.705259778 upper=2.705259778 effort=11.6 velocity=40
- joint thigh_fr_to_knee_fr_j: limit lower=-2.705259778 upper=2.705259778 -> lower=-2.705259778 upper=2.705259778 effort=11.6 velocity=40
- joint thigh_hl_to_knee_hl_j: limit lower=-2.705259778 upper=2.705259778 -> lower=-2.705259778 upper=2.705259778 effort=11.6 velocity=40
- joint thigh_hr_to_knee_hr_j: limit lower=-2.705259778 upper=2.705259778 -> lower=-2.705259778 upper=2.705259778 effort=11.6 velocity=40
- joint torso_to_abduct_fl_j: limit lower=-2.094395102 upper=2.094395102 velocity=40 -> lower=-2.094395102 upper=2.094395102 effort=18 velocity=40
- joint torso_to_abduct_fr_j: limit lower=-2.094395102 upper=2.094395102 velocity=40 -> lower=-2.094395102 upper=2.094395102 effort=18 velocity=40
- joint torso_to_abduct_hl_j: limit lower=-2.094395102 upper=2.094395102 velocity=40 -> lower=-2.094395102 upper=2.094395102 effort=18 velocity=40
- joint torso_to_abduct_hr_j: limit lower=-2.094395102 upper=2.094395102 velocity=40 -> lower=-2.094395102 upper=2.094395102 effort=18 velocity=40

File: rsc/mini_cheetah/otherVersions/mini-cheetah-vision-cont.urdf (robot description, URDF)
Before this commit: robot mini_cheetah, 17 links, 16 joints
Links:
- link toe_fl: mass 0.0 -> 0.15
- link toe_fr: mass 0.0 -> 0.15
- link toe_hl: mass 0.0 -> 0.15
- link toe_hr: mass 0.0 -> 0.15
Joints:
- joint abduct_fl_to_thigh_fl_j: limit lower=-2.356194 upper=2.356194 velocity=40 -> (none); type revolute -> continuous
- joint abduct_fr_to_thigh_fr_j: limit lower=-2.356194 upper=2.356194 velocity=40 -> (none); type revolute -> continuous
- joint abduct_hl_to_thigh_hl_j: limit lower=-2.356194 upper=2.356194 velocity=40 -> (none); type revolute -> continuous
- joint abduct_hr_to_thigh_hr_j: limit lower=-2.356194 upper=2.356194 velocity=40 -> (none); type revolute -> continuous
- joint thigh_fl_to_knee_fl_j: limit lower=-1.352629889 upper=1.352629889 -> (none); type revolute -> continuous
- joint thigh_fr_to_knee_fr_j: limit lower=-1.352629889 upper=1.352629889 -> (none); type revolute -> continuous
- joint thigh_hl_to_knee_hl_j: limit lower=-1.352629889 upper=1.352629889 -> (none); type revolute -> continuous
- joint thigh_hr_to_knee_hr_j: limit lower=-1.352629889 upper=1.352629889 -> (none); type revolute -> continuous
- joint torso_to_abduct_fl_j: limit lower=-1.0471975512 upper=1.0471975512 velocity=40 -> (none); type revolute -> continuous
- joint torso_to_abduct_fr_j: limit lower=-1.0471975512 upper=1.0471975512 velocity=40 -> (none); type revolute -> continuous
- joint torso_to_abduct_hl_j: limit lower=-1.0471975512 upper=1.0471975512 velocity=40 -> (none); type revolute -> continuous
- joint torso_to_abduct_hr_j: limit lower=-1.0471975512 upper=1.0471975512 velocity=40 -> (none); type revolute -> continuous

File: rsc/mini_cheetah/otherVersions/mini-cheetah-vision-original.urdf (robot description, URDF)
Before this commit: robot mini_cheetah, 17 links, 16 joints
Links:
- removed link toe_fl
- removed link toe_fr
- removed link toe_hl
- removed link toe_hr
- link abduct_fl: geometry collision mesh filename=meshes/mini_abad.obj; visual mesh filename=meshes/mini_abad.obj
- link abduct_fr: geometry collision mesh filename=meshes/mini_abad.obj; visual mesh filename=meshes/mini_abad.obj
- link abduct_hl: geometry collision mesh filename=meshes/mini_abad.obj; visual mesh filename=meshes/mini_abad.obj
- link abduct_hr: geometry collision mesh filename=meshes/mini_abad.obj; visual mesh filename=meshes/mini_abad.obj
- link body: geometry collision mesh filename=meshes/mini_body.obj; visual mesh filename=meshes/mini_body.obj
- link shank_fl: geometry collision mesh filename=meshes/mini_lower_link.obj; visual mesh filename=meshes/mini_lower_link.obj
- link shank_fr: geometry collision mesh filename=meshes/mini_lower_link.obj; visual mesh filename=meshes/mini_lower_link.obj
- link shank_hl: geometry collision mesh filename=meshes/mini_lower_link.obj; visual mesh filename=meshes/mini_lower_link.obj
- link shank_hr: geometry collision mesh filename=meshes/mini_lower_link.obj; visual mesh filename=meshes/mini_lower_link.obj
- link thigh_fl: geometry collision mesh filename=meshes/mini_upper_link.obj; visual mesh filename=meshes/mini_upper_link.obj
- link thigh_fr: geometry collision mesh filename=meshes/mini_upper_link.obj; visual mesh filename=meshes/mini_upper_link.obj
- link thigh_hl: geometry collision mesh filename=meshes/mini_upper_link.obj; visual mesh filename=meshes/mini_upper_link.obj
- link thigh_hr: geometry collision mesh filename=meshes/mini_upper_link.obj; visual mesh filename=meshes/mini_upper_link.obj
Joints:
- removed joint toe_fl_joint
- removed joint toe_fr_joint
- removed joint toe_hl_joint
- removed joint toe_hr_joint
- joint abduct_fl_to_thigh_fl_j: limit lower=-2.356194 upper=2.356194 velocity=40 -> (none); type revolute -> continuous
- joint abduct_fr_to_thigh_fr_j: limit lower=-2.356194 upper=2.356194 velocity=40 -> (none); type revolute -> continuous
- joint abduct_hl_to_thigh_hl_j: limit lower=-2.356194 upper=2.356194 velocity=40 -> (none); type revolute -> continuous
- joint abduct_hr_to_thigh_hr_j: limit lower=-2.356194 upper=2.356194 velocity=40 -> (none); type revolute -> continuous
- joint thigh_fl_to_knee_fl_j: limit lower=-1.352629889 upper=1.352629889 -> (none); type revolute -> continuous
- joint thigh_fr_to_knee_fr_j: limit lower=-1.352629889 upper=1.352629889 -> (none); type revolute -> continuous
- joint thigh_hl_to_knee_hl_j: limit lower=-1.352629889 upper=1.352629889 -> (none); type revolute -> continuous
- joint thigh_hr_to_knee_hr_j: limit lower=-1.352629889 upper=1.352629889 -> (none); type revolute -> continuous
- joint torso_to_abduct_fl_j: limit lower=-1.0471975512 upper=1.0471975512 velocity=40 -> (none); type revolute -> continuous
- joint torso_to_abduct_fr_j: limit lower=-1.0471975512 upper=1.0471975512 velocity=40 -> (none); type revolute -> continuous
- joint torso_to_abduct_hl_j: limit lower=-1.0471975512 upper=1.0471975512 velocity=40 -> (none); type revolute -> continuous
- joint torso_to_abduct_hr_j: limit lower=-1.0471975512 upper=1.0471975512 velocity=40 -> (none); origin xyz=-0.2 -0.049 0.0 rpy=0 0 0 -> xyz=0.2 -0.049 0.0 rpy=0 0 0; type revolute -> continuous

Commit message: urdf body collision box is made smaller, obs noise function is added

File: rsc/mini_cheetah/mini-cheetah-vision-v1.3.urdf (robot description, URDF)
Before this commit: robot mini_cheetah, 17 links, 16 joints
Links:
- link body: geometry collision box size=0.244 0.18 0.044; visual mesh filename=meshes/mini_body.obj

Commit message: Initial pose randomization, Observation noise, Airtime reward, urdf joint limit modified, control_dt: 500Hz.

File: rsc/mini_cheetah/mini-cheetah-vision-v1.3.urdf (robot description, URDF)
Before this commit: robot mini_cheetah, 17 links, 16 joints
Links:
- link shank_fr: geometry collision box size=0.016 0.016 0.175; visual mesh filename=meshes/mini_lower_link.obj
Joints:
- joint abduct_fl_to_thigh_fl_j: limit lower=-4.712388 upper=4.712388 effort=18 velocity=40 -> lower=-5. upper=5. effort=18 velocity=40
- joint abduct_fr_to_thigh_fr_j: limit lower=-4.712388 upper=4.712388 effort=18 velocity=40 -> lower=-5. upper=5. effort=18 velocity=40
- joint abduct_hl_to_thigh_hl_j: limit lower=-4.712388 upper=4.712388 effort=18 velocity=40 -> lower=-5. upper=5. effort=18 velocity=40
- joint abduct_hr_to_thigh_hr_j: limit lower=-4.712388 upper=4.712388 effort=18 velocity=40 -> lower=-5. upper=5. effort=18 velocity=40
- joint torso_to_abduct_fl_j: limit lower=-2.094395102 upper=2.094395102 effort=18 velocity=40 -> lower=-1.5 upper=1.5 effort=18 velocity=40
- joint torso_to_abduct_fr_j: limit lower=-2.094395102 upper=2.094395102 effort=18 velocity=40 -> lower=-1.5 upper=1.5 effort=18 velocity=40
- joint torso_to_abduct_hl_j: limit lower=-2.094395102 upper=2.094395102 effort=18 velocity=40 -> lower=-1.5 upper=1.5 effort=18 velocity=40
- joint torso_to_abduct_hr_j: limit lower=-2.094395102 upper=2.094395102 effort=18 velocity=40 -> lower=-1.5 upper=1.5 effort=18 velocity=40

Commit message: stepdata error correction, urdf collision box size modified, gamma: 0.996->0.98

File: rsc/mini_cheetah/mini-cheetah-vision-v1.3.urdf (robot description, URDF)
Before this commit: robot mini_cheetah, 17 links, 16 joints
Links:
- link shank_fl: geometry collision box size=0.016 0.016 0.16; visual mesh filename=meshes/mini_lower_link.obj
- link shank_fr: geometry collision box size=0.016 0.016 0.16; visual mesh filename=meshes/mini_lower_link.obj
- link shank_hl: geometry collision box size=0.016 0.016 0.16; visual mesh filename=meshes/mini_lower_link.obj
- link shank_hr: geometry collision box size=0.016 0.016 0.16; visual mesh filename=meshes/mini_lower_link.obj
- link thigh_fl: geometry collision box size=0.025 0.025 0.22; visual mesh filename=meshes/mini_upper_link.obj
- link thigh_fr: geometry collision box size=0.025 0.025 0.22; visual mesh filename=meshes/mini_upper_link.obj
- link thigh_hl: geometry collision box size=0.025 0.025 0.22; visual mesh filename=meshes/mini_upper_link.obj
- link thigh_hr: geometry collision box size=0.025 0.025 0.22; visual mesh filename=meshes/mini_upper_link.obj

Commit message: order of update: modified, reward coeff: modified, urdf: size modified

File: rsc/mini_cheetah/mini-cheetah-vision-v1.3.urdf (robot description, URDF)
Before this commit: robot mini_cheetah, 17 links, 16 joints
Joints:
- joint abduct_fl_to_thigh_fl_j: origin xyz=0.0 0.062 0.00 rpy=0.0 0.0 0.0 -> xyz=0.055 0.019 0.00 rpy=0.0 0.0 0.0
- joint abduct_fr_to_thigh_fr_j: origin xyz=0.0 -0.062 0.00 rpy=0.0 0.0 0.0 -> xyz=0.055 -0.019 0.00 rpy=0.0 0.0 0.0
- joint abduct_hl_to_thigh_hl_j: origin xyz=0.0 0.062 0.00 rpy=0.0 0.0 0.0 -> xyz=0.055 0.019 0.00 rpy=0.0 3.141592 0.0
- joint abduct_hr_to_thigh_hr_j: origin xyz=0.0 -0.062 0.00 rpy=0.0 0.0 0.0 -> xyz=0.055 -0.019 0.00 rpy=0.0 3.141592 0.0
- joint thigh_fl_to_knee_fl_j: origin xyz=0.0 0.0 -0.209 rpy=0.0 0 0.0 -> xyz=0.0 0.049 -0.2085 rpy=0.0 0 0.0
- joint thigh_fr_to_knee_fr_j: origin xyz=0.0 0.0 -0.209 rpy=0.0 0 0.0 -> xyz=0.0 -0.049 -0.2085 rpy=0.0 0 0.0
- joint thigh_hl_to_knee_hl_j: origin xyz=0.0 0.0 -0.209 rpy=0.0 0 0.0 -> xyz=0.0 0.049 -0.2085 rpy=0.0 0 0.0
- joint thigh_hr_to_knee_hr_j: origin xyz=0.0 0.0 -0.209 rpy=0.0 0 0.0 -> xyz=0.0 -0.049 -0.2085 rpy=0.0 0 0.0
- joint toe_fl_joint: origin xyz=0 0 -0.18 -> xyz=0 0 -0.1885
- joint toe_fr_joint: origin xyz=0 0 -0.18 -> xyz=0 0 -0.1885
- joint toe_hl_joint: origin xyz=0 0 -0.18 -> xyz=0 0 -0.1885
- joint toe_hr_joint: origin xyz=0 0 -0.18 -> xyz=0 0 -0.1885
- joint torso_to_abduct_fl_j: origin xyz=0.20 0.049 0.0 rpy=0 0 0 -> xyz=0.14775 0.049 0.0 rpy=0 0 0
- joint torso_to_abduct_fr_j: origin xyz=0.2 -0.049 0.0 rpy=0 0 0 -> xyz=0.14775 -0.049 0.0 rpy=0 0 0
- joint torso_to_abduct_hl_j: origin xyz=-0.2 0.049 0.0 rpy=0 0 0 -> xyz=-0.14775 0.049 0.0 rpy=0 3.141592 0
- joint torso_to_abduct_hr_j: origin xyz=-0.2 -0.049 0.0 rpy=0 0 0 -> xyz=-0.14775 -0.049 0.0 rpy=0 3.141592 0

File: rsc/mini_cheetah/otherVersions/mini-cheetah-vision.urdf (robot description, URDF)
Before this commit: robot mini_cheetah, 17 links, 16 joints
Links:
- removed link toe_fl
- removed link toe_fr
- removed link toe_hl
- removed link toe_hr
- link abduct_fl: geometry collision mesh filename=meshes/mini_vision_abd.dae; visual mesh filename=meshes/mini_vision_abd.dae
- link abduct_fr: geometry collision mesh filename=meshes/mini_vision_abd.dae; visual mesh filename=meshes/mini_vision_abd.dae
- link abduct_hl: geometry collision mesh filename=meshes/mini_vision_abd.dae; visual mesh filename=meshes/mini_vision_abd.dae
- link abduct_hr: geometry collision mesh filename=meshes/mini_vision_abd.dae; visual mesh filename=meshes/mini_vision_abd.dae
- link body: geometry collision mesh filename=meshes/mini_vision_body.dae; visual mesh filename=meshes/mini_vision_body.dae
- link shank_fl: geometry collision mesh filename=meshes/lower_leg.dae; visual mesh filename=meshes/lower_leg.dae
- link shank_fr: geometry collision mesh filename=meshes/lower_leg.dae; visual mesh filename=meshes/lower_leg.dae
- link shank_hl: geometry collision mesh filename=meshes/lower_leg.dae; visual mesh filename=meshes/lower_leg.dae
- link shank_hr: geometry collision mesh filename=meshes/lower_leg.dae; visual mesh filename=meshes/lower_leg.dae
- link thigh_fl: geometry collision mesh filename=meshes/mini_vision_upper_leg.dae; visual mesh filename=meshes/mini_vision_upper_leg.dae
- link thigh_fr: geometry collision mesh filename=meshes/mini_vision_upper_leg.dae; visual mesh filename=meshes/mini_vision_upper_leg.dae
- link thigh_hl: geometry collision mesh filename=meshes/mini_vision_upper_leg.dae; visual mesh filename=meshes/mini_vision_upper_leg.dae
- link thigh_hr: geometry collision mesh filename=meshes/mini_vision_upper_leg.dae; visual mesh filename=meshes/mini_vision_upper_leg.dae
Joints:
- removed joint toe_fl_joint
- removed joint toe_fr_joint
- removed joint toe_hl_joint
- removed joint toe_hr_joint
- joint abduct_fl_to_thigh_fl_j: limit lower=-2.356194 upper=2.356194 velocity=40 -> (none); origin xyz=0.0 0.062 0.00 rpy=0.0 0.0 0.0 -> xyz=0.055 0.019 0.00 rpy=0.0 0.0 0.0; type revolute -> continuous
- joint abduct_fr_to_thigh_fr_j: limit lower=-2.356194 upper=2.356194 velocity=40 -> (none); origin xyz=0.0 -0.062 0.00 rpy=0.0 0.0 0.0 -> xyz=0.055 -0.019 0.00 rpy=0.0 0.0 0.0; type revolute -> continuous
- joint abduct_hl_to_thigh_hl_j: limit lower=-2.356194 upper=2.356194 velocity=40 -> (none); origin xyz=0.0 0.062 0.00 rpy=0.0 0.0 0.0 -> xyz=0.055 0.019 0.00 rpy=0.0 3.141592 0.0; type revolute -> continuous
- joint abduct_hr_to_thigh_hr_j: limit lower=-2.356194 upper=2.356194 velocity=40 -> (none); origin xyz=0.0 -0.062 0.00 rpy=0.0 0.0 0.0 -> xyz=0.055 -0.019 0.00 rpy=0.0 3.141592 0.0; type revolute -> continuous
- joint thigh_fl_to_knee_fl_j: limit lower=-1.352629889 upper=1.352629889 -> (none); origin xyz=0.0 0.0 -0.209 rpy=0.0 0 0.0 -> xyz=0.0 0.049 -0.2085 rpy=0.0 0 0.0; type revolute -> continuous
- joint thigh_fr_to_knee_fr_j: limit lower=-1.352629889 upper=1.352629889 -> (none); origin xyz=0.0 0.0 -0.209 rpy=0.0 0 0.0 -> xyz=0.0 -0.049 -0.2085 rpy=0.0 0 0.0; type revolute -> continuous
- joint thigh_hl_to_knee_hl_j: limit lower=-1.352629889 upper=1.352629889 -> (none); origin xyz=0.0 0.0 -0.209 rpy=0.0 0 0.0 -> xyz=0.0 0.049 -0.2085 rpy=0.0 0 0.0; type revolute -> continuous
- joint thigh_hr_to_knee_hr_j: limit lower=-1.352629889 upper=1.352629889 -> (none); origin xyz=0.0 0.0 -0.209 rpy=0.0 0 0.0 -> xyz=0.0 -0.049 -0.2085 rpy=0.0 0 0.0; type revolute -> continuous
- joint torso_to_abduct_fl_j: limit lower=-1.0471975512 upper=1.0471975512 velocity=40 -> (none); origin xyz=0.20 0.049 0.0 rpy=0 0 0 -> xyz=0.14775 0.049 0.0 rpy=0 0 0; type revolute -> continuous
- joint torso_to_abduct_fr_j: limit lower=-1.0471975512 upper=1.0471975512 velocity=40 -> (none); origin xyz=0.2 -0.049 0.0 rpy=0 0 0 -> xyz=0.14775 -0.049 0.0 rpy=0 0 0; type revolute -> continuous
- joint torso_to_abduct_hl_j: limit lower=-1.0471975512 upper=1.0471975512 velocity=40 -> (none); origin xyz=-0.2 0.049 0.0 rpy=0 0 0 -> xyz=-0.14775 0.049 0.0 rpy=0 3.141592 0; type revolute -> continuous
- joint torso_to_abduct_hr_j: limit lower=-1.0471975512 upper=1.0471975512 velocity=40 -> (none); origin xyz=-0.2 -0.049 0.0 rpy=0 0 0 -> xyz=-0.14775 -0.049 0.0 rpy=0 3.141592 0; type revolute -> continuous

Commit message: change: urdf knee size.

File: rsc/mini_cheetah/mini-cheetah-vision-v1.3.urdf (robot description, URDF)
Before this commit: robot mini_cheetah, 17 links, 16 joints
Links:
- link toe_fl: geometry collision sphere radius=0.02
- link toe_fr: geometry collision sphere radius=0.02
- link toe_hl: geometry collision sphere radius=0.02
- link toe_hr: geometry collision sphere radius=0.02
Joints:
- joint toe_fl_joint: origin xyz=0 0 -0.1885 -> xyz=0 0 -0.175
- joint toe_fr_joint: origin xyz=0 0 -0.1885 -> xyz=0 0 -0.175
- joint toe_hl_joint: origin xyz=0 0 -0.1885 -> xyz=0 0 -0.175
- joint toe_hr_joint: origin xyz=0 0 -0.1885 -> xyz=0 0 -0.175

Commit message: change: urdf frame, more detailed obs noise

File: rsc/mini_cheetah/mini-cheetah-vision-v1.3.urdf (robot description, URDF)
Before this commit: robot mini_cheetah, 17 links, 16 joints
Links:
- link shank_fl: geometry collision box size=0.012 0.012 0.195; visual mesh filename=meshes/mini_lower_link.obj
- link shank_fr: geometry collision box size=0.012 0.012 0.195; visual mesh filename=meshes/mini_lower_link.obj
- link shank_hl: geometry collision box size=0.012 0.012 0.195; visual mesh filename=meshes/mini_lower_link.obj
- link shank_hr: geometry collision box size=0.012 0.012 0.195; visual mesh filename=meshes/mini_lower_link.obj
- link toe_fl: geometry collision sphere radius=0.0
- link toe_fr: geometry collision sphere radius=0.0
- link toe_hl: geometry collision sphere radius=0.0
- link toe_hr: geometry collision sphere radius=0.0
Joints:
- joint abduct_fl_to_thigh_fl_j: origin xyz=0.055 0.019 0.00 rpy=0.0 0.0 0.0 -> xyz=0.0 0.019 0.00 rpy=0.0 0.0 0.0
- joint abduct_fr_to_thigh_fr_j: origin xyz=0.055 -0.019 0.00 rpy=0.0 0.0 0.0 -> xyz=0.0 -0.019 0.00 rpy=0.0 0.0 0.0
- joint abduct_hl_to_thigh_hl_j: origin xyz=0.055 0.019 0.00 rpy=0.0 3.141592 0.0 -> xyz=-0.0 0.019 0.00 rpy=0.0 0 0.0
- joint abduct_hr_to_thigh_hr_j: origin xyz=0.055 -0.019 0.00 rpy=0.0 3.141592 0.0 -> xyz=-0.0 -0.019 0.00 rpy=0.0 0 0.0
- joint toe_fl_joint: origin xyz=0 0 -0.175 -> xyz=0 0 -0.195
- joint toe_fr_joint: origin xyz=0 0 -0.175 -> xyz=0 0 -0.195
- joint toe_hl_joint: origin xyz=0 0 -0.175 -> xyz=0 0 -0.195
- joint toe_hr_joint: origin xyz=0 0 -0.175 -> xyz=0 0 -0.195
- joint torso_to_abduct_fl_j: origin xyz=0.14775 0.049 0.0 rpy=0 0 0 -> xyz=0.20275 0.049 0.0 rpy=0 0 0
- joint torso_to_abduct_fr_j: origin xyz=0.14775 -0.049 0.0 rpy=0 0 0 -> xyz=0.20275 -0.049 0.0 rpy=0 0 0
- joint torso_to_abduct_hl_j: origin xyz=-0.14775 0.049 0.0 rpy=0 3.141592 0 -> xyz=-0.20275 0.049 0.0 rpy=0 0 0
- joint torso_to_abduct_hr_j: origin xyz=-0.14775 -0.049 0.0 rpy=0 3.141592 0 -> xyz=-0.20275 -0.049 0.0 rpy=0 0 0

Commit message: urdf: intertial change, rotor. PGain: 50->30. actionStd: 0.3->0.1. sim_dt: 0.002->0.001. control_dt: 0.016->0.02. reward coefficient change.

File: rsc/mini_cheetah/mini-cheetah-vision-v1.3.urdf (robot description, URDF)
Before this commit: robot mini_cheetah, 17 links, 16 joints
Links:
- added link abduct_fl_rotor, mass 0.055
- added link abduct_fr_rotor, mass 0.055
- added link abduct_hl_rotor, mass 0.055
- added link abduct_hr_rotor, mass 0.055
- added link shank_fl_rotor, mass 0.055
- added link shank_fr_rotor, mass 0.055
- added link shank_hl_rotor, mass 0.055
- added link shank_hr_rotor, mass 0.055
- added link thigh_fl_rotor, mass 0.055
- added link thigh_fr_rotor, mass 0.055
- added link thigh_hl_rotor, mass 0.055
- added link thigh_hr_rotor, mass 0.055
- link body: mass 5.868 -> 5.208
- link toe_fl: geometry collision sphere radius=0.018
- link toe_fr: geometry collision sphere radius=0.018
- link toe_hl: geometry collision sphere radius=0.018
- link toe_hr: geometry collision sphere radius=0.018
Joints:
- added joint abduct_fl_rotor_j: type fixed, parent abduct_fl, child abduct_fl_rotor, origin xyz=-0.055 0 0
- added joint abduct_fr_rotor_j: type fixed, parent abduct_fr, child abduct_fr_rotor, origin xyz=-0.055 0 0
- added joint abduct_hl_rotor_j: type fixed, parent abduct_hl, child abduct_hl_rotor, origin xyz=0.055 0 0
- added joint abduct_hr_rotor_j: type fixed, parent abduct_hr, child abduct_hr_rotor, origin xyz=0.055 0 0
- added joint shank_fl_rotor_j: type fixed, parent shank_fl, child shank_fl_rotor, origin xyz=0 0 0
- added joint shank_fr_rotor_j: type fixed, parent shank_fr, child shank_fr_rotor, origin xyz=0 0 0
- added joint shank_hl_rotor_j: type fixed, parent shank_hl, child shank_hl_rotor, origin xyz=0 0 0
- added joint shank_hr_rotor_j: type fixed, parent shank_hr, child shank_hr_rotor, origin xyz=0 0 0
- added joint thigh_fl_rotor_j: type fixed, parent thigh_fl, child thigh_fl_rotor, origin xyz=0 0 0
- added joint thigh_fr_rotor_j: type fixed, parent thigh_fr, child thigh_fr_rotor, origin xyz=0 0 0
- added joint thigh_hl_rotor_j: type fixed, parent thigh_hl, child thigh_hl_rotor, origin xyz=0 0 0
- added joint thigh_hr_rotor_j: type fixed, parent thigh_hr, child thigh_hr_rotor, origin xyz=0 0 0
