Commit message: modified: urdf com, rotor inertia.

File: rsc/mini_cheetah/mini-cheetah-vision-v1.3.urdf (robot description, URDF)
Before this commit: robot mini_cheetah, 29 links, 28 joints
Joints:
- joint abduct_fl_rotor_j: origin xyz=-0.055 0 0 -> xyz=0 0 0
- joint abduct_fl_to_thigh_fl_j: limit lower=-5. upper=5. effort=18 velocity=40 -> lower=-5. upper=5. effort=17 velocity=40; origin xyz=0.0 0.019 0.00 rpy=0.0 0.0 0.0 -> xyz=0.055 0.019 0.00 rpy=0.0 0.0 0.0
- joint abduct_fr_rotor_j: origin xyz=-0.055 0 0 -> xyz=0 0 0
- joint abduct_fr_to_thigh_fr_j: limit lower=-5. upper=5. effort=18 velocity=40 -> lower=-5. upper=5. effort=17 velocity=40; origin xyz=0.0 -0.019 0.00 rpy=0.0 0.0 0.0 -> xyz=0.055 -0.019 0.00 rpy=0.0 0.0 0.0
- joint abduct_hl_rotor_j: origin xyz=0.055 0 0 -> xyz=0.0 0 0
- joint abduct_hl_to_thigh_hl_j: limit lower=-5. upper=5. effort=18 velocity=40 -> lower=-5. upper=5. effort=17 velocity=40; origin xyz=-0.0 0.019 0.00 rpy=0.0 0 0.0 -> xyz=-0.055 0.019 0.00 rpy=0.0 0 0.0
- joint abduct_hr_rotor_j: origin xyz=0.055 0 0 -> xyz=0. 0 0
- joint abduct_hr_to_thigh_hr_j: limit lower=-5. upper=5. effort=18 velocity=40 -> lower=-5. upper=5. effort=17 velocity=40; origin xyz=-0.0 -0.019 0.00 rpy=0.0 0 0.0 -> xyz=-0.055 -0.019 0.00 rpy=0.0 0 0.0
- joint thigh_fl_to_knee_fl_j: limit lower=-2.705259778 upper=2.705259778 effort=11.6 velocity=40 -> lower=-2.705259778 upper=2.705259778 effort=26 velocity=40
- joint thigh_fr_to_knee_fr_j: limit lower=-2.705259778 upper=2.705259778 effort=11.6 velocity=40 -> lower=-2.705259778 upper=2.705259778 effort=26 velocity=40
- joint thigh_hl_to_knee_hl_j: limit lower=-2.705259778 upper=2.705259778 effort=11.6 velocity=40 -> lower=-2.705259778 upper=2.705259778 effort=26 velocity=40
- joint thigh_hr_to_knee_hr_j: limit lower=-2.705259778 upper=2.705259778 effort=11.6 velocity=40 -> lower=-2.705259778 upper=2.705259778 effort=26 velocity=40
- joint torso_to_abduct_fl_j: limit lower=-1.5 upper=1.5 effort=18 velocity=40 -> lower=-1.5 upper=1.5 effort=17 velocity=40; origin xyz=0.20275 0.049 0.0 rpy=0 0 0 -> xyz=0.14775 0.049 0.0 rpy=0 0 0
- joint torso_to_abduct_fr_j: limit lower=-1.5 upper=1.5 effort=18 velocity=40 -> lower=-1.5 upper=1.5 effort=17 velocity=40; origin xyz=0.20275 -0.049 0.0 rpy=0 0 0 -> xyz=0.14775 -0.049 0.0 rpy=0 0 0
- joint torso_to_abduct_hl_j: limit lower=-1.5 upper=1.5 effort=18 velocity=40 -> lower=-1.5 upper=1.5 effort=17 velocity=40; origin xyz=-0.20275 0.049 0.0 rpy=0 0 0 -> xyz=-0.14775 0.049 0.0 rpy=0 0 0
- joint torso_to_abduct_hr_j: limit lower=-1.5 upper=1.5 effort=18 velocity=40 -> lower=-1.5 upper=1.5 effort=17 velocity=40; origin xyz=-0.20275 -0.049 0.0 rpy=0 0 0 -> xyz=-0.14775 -0.049 0.0 rpy=0 0 0

Commit message: On debugging: same mass matrix as in Cheetah Software.

File: rsc/mini_cheetah/mini-cheetah-vision-v1.3.urdf (robot description, URDF)
Before this commit: robot mini_cheetah, 29 links, 28 joints
Links:
- link abduct_fl: geometry collision cylinder length=0.022 radius=0.048; visual mesh filename=meshes/mini_vision_abd.dae
- link body: geometry collision box size=0.244 0.18 0.044; visual mesh filename=meshes/mini_vision_body.dae
- link shank_fl: geometry collision box size=0.012 0.012 0.195; visual mesh filename=meshes/lower_leg.dae
- link thigh_fl: geometry collision box size=0.025 0.025 0.22; visual mesh filename=meshes/mini_vision_upper_leg.dae
Joints:
- joint shank_fl_rotor_j: origin xyz=0 0 0 -> xyz=0 0.049 0; parent shank_fl -> thigh_fl
- joint shank_fr_rotor_j: parent shank_fr -> thigh_fr
- joint shank_hl_rotor_j: origin xyz=0 0 0 -> xyz=0 0.049 0; parent shank_hl -> thigh_hl
- joint shank_hr_rotor_j: origin xyz=0 0 0 -> xyz=0 -0.049 0; parent shank_hr -> thigh_hr

Commit message: On debugging: COM, rotor.

File: rsc/mini_cheetah/mini-cheetah-vision-v1.3.urdf (robot description, URDF)
Before this commit: robot mini_cheetah, 29 links, 28 joints
Joints:
- joint abduct_fl_rotor_j: origin xyz=0 0 0 -> xyz=0.14775 0.049 0.0; parent abduct_fl -> body
- joint abduct_fr_rotor_j: origin xyz=0 0 0 -> xyz=0.14775 -0.049 0.0; parent abduct_fr -> body
- joint abduct_hl_rotor_j: origin xyz=0.0 0 0 -> xyz=-0.14775 0.049 0.0; parent abduct_hl -> body
- joint abduct_hr_rotor_j: origin xyz=0. 0 0 -> xyz=-0.14775 -0.049 0.0; parent abduct_hr -> body
- joint shank_fr_rotor_j: origin xyz=0 0 0 -> xyz=0.0 -0.049 0.0
- joint thigh_fl_rotor_j: origin xyz=0 0 0 -> xyz=0.055 0.019 0.00; parent thigh_fl -> abduct_fl
- joint thigh_fr_rotor_j: origin xyz=0 0 0 -> xyz=0.055 -0.019 0.00; parent thigh_fr -> abduct_fr
- joint thigh_hl_rotor_j: origin xyz=0 0 0 -> xyz=-0.055 0.019 0.00; parent thigh_hl -> abduct_hl
- joint thigh_hr_rotor_j: origin xyz=0 0 0 -> xyz=-0.055 -0.019 0.00; parent thigh_hr -> abduct_hr

Commit message: modified: control_dt 50Hz, nominal pose, standing command, forward max 1.5m/s, footClearance 0.1m, airtime 0.5s->0.4s, urdf: foot ball size 0.018->0.01

File: rsc/mini_cheetah/mini-cheetah-vision-v1.3.urdf (robot description, URDF)
Before this commit: robot mini_cheetah, 29 links, 28 joints
Links:
- link abduct_fl: geometry collision cylinder length=0.022 radius=0.048; visual mesh filename=meshes/mini_abad.obj
- link shank_fl: geometry collision box size=0.012 0.012 0.195; visual mesh filename=meshes/mini_lower_link.obj
- link thigh_fl: geometry collision box size=0.025 0.025 0.22; visual mesh filename=meshes/mini_upper_link.obj
- link toe_fl: geometry collision sphere radius=0.01
- link toe_fr: geometry collision sphere radius=0.01
- link toe_hl: geometry collision sphere radius=0.01
- link toe_hr: geometry collision sphere radius=0.01

Commit message: modified: kp20 kd04, higher init noise, higher smoothness coeff, bigger foot ball.

File: rsc/mini_cheetah/mini-cheetah-vision-v1.3.urdf (robot description, URDF)
Before this commit: robot mini_cheetah, 29 links, 28 joints
Links:
- link toe_fl: geometry collision sphere radius=0.013
- link toe_fr: geometry collision sphere radius=0.013
- link toe_hl: geometry collision sphere radius=0.013
- link toe_hr: geometry collision sphere radius=0.013
