Commit message: modified: urdf

File: rsc/mini_cheetah/mini-cheetah-vision-v1.5.urdf (robot description, URDF)
Before this commit: robot mini_cheetah, 29 links, 28 joints
Links:
- link body: mass 5.208 -> 4.832
- link shank_fl: mass 0.064 -> 0.158
- link shank_fr: mass 0.064 -> 0.158
- link shank_hl: mass 0.064 -> 0.158
- link shank_hr: mass 0.064 -> 0.158

Commit message: Very Fast Learning. added: entropy coeff, foot collision randomization. modified: minibatch, lr scheduler, curriculum factor, foot clearance, ground friction 0.4, body height observation.

File: rsc/mini_cheetah/mini-cheetah-vision-v1.5.urdf (robot description, URDF)
Before this commit: robot mini_cheetah, 29 links, 28 joints
Links:
- link toe_fl: geometry collision sphere radius=0.018
- link toe_fr: geometry collision sphere radius=0.018
- link toe_hl: geometry collision sphere radius=0.018
- link toe_hr: geometry collision sphere radius=0.018
